File: KiCad/Protection_Catapult_PCB/_autosave-Protection_Catapult_PCB.kicad_pcb (KiCad board)
At the start: 2 copper layers, 160 x 100 mm, 35 parts, among them J1 Motor_I, J10 Screw_Terminal_01x03, J11 Motor NEMA I, J12 Motor DC, J13 Motores 28BYJ-48, J15 Servo, J16 Motor NEMA D, J2 Motor_D, J3 Control_D, J4 Control_I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

Commit message: Inventor and PCB Update. Full program started.
Parts:
- removed U6: ESP32-S3-DevKitC, PCM_Espressif:ESP32-S3-DevKitC
- added J14: Screw_Terminal_01x09, Connector_PinHeader_2.54mm:PinHeader_1x09_P2.54mm_Vertical, F.Cu at (160.0, 48.3)
- added J17: Motor, Connector_JST:JST_XH_B2B-XH-A_1x02_P2.50mm_Vertical, F.Cu at (119.4, 137.2)
- added J18: Screw_Terminal_01x09, Connector_PinHeader_2.54mm:PinHeader_1x09_P2.54mm_Vertical, F.Cu at (175.3, 48.3)
- J10: value Screw_Terminal_01x03 -> Servo
- J12: footprint Connector_JST:JST_XH_B2B-XH-A_1x02_P2.50mm_Vertical -> Connector_JST:JST_XH_B4B-XH-A_1x04_P2.50mm_Vertical
- J15: value Servo -> Final carrera; footprint Connector_JST:JST_XH_B1B-XH-AM_1x01_P2.50mm_Vertical -> Connector_JST:JST_XH_B2B-XH-A_1x02_P2.50mm_Vertical
- moved J15 56.5 mm to (157.5, 76.2), turned to 180 degrees
- moved J13 41.4 mm to (172.6, 76.2), turned to 180 degrees
- moved J12 35.8 mm to (185.4, 78.7), turned to 90 degrees
- moved J11 28.7 mm to (185.4, 53.3), turned to 90 degrees
- moved J16 28.4 mm to (185.4, 63.5), turned to 90 degrees
Connections:
- J10 pad 1: /Servo -> /IO6
- J11 pad 1: Net-(J11-Pin_1) -> /IO12
- J11 pad 2: Net-(J11-Pin_2) -> /IO13
- J12 pad 1: Net-(J12-Pin_1) -> GND
- J12 pad 2: Net-(J12-Pin_2) -> /IO8
- J13 pad 1: Net-(J13-Pin_1) -> /IO2
- J13 pad 2: Net-(J13-Pin_2) -> /IO3
- J13 pad 3: Net-(J13-Pin_3) -> /IO4
- J13 pad 4: Net-(J13-Pin_4) -> /IO5
- J15 pad 1: Net-(J15-Pin_1) -> GND
- J16 pad 1: Net-(J16-Pin_1) -> /IO10
- J16 pad 2: Net-(J16-Pin_2) -> /IO11
Routing:
- net GND: track 322.7 -> 409.2 mm
- net +5V: track 195.8 -> 277.1 mm, vias 6 -> 16
- net /IO2: track 0.00 -> 33.1 mm
- net /IO3: track 0.00 -> 28.0 mm
- net /IO4: track 0.00 -> 22.9 mm
- net /IO9: track 0.00 -> 17.9 mm
- net /IO8: track 0.00 -> 17.8 mm
- net /IO5: track 0.00 -> 17.8 mm
- net /IO12: track 0.00 -> 15.2 mm
- net /IO13: track 0.00 -> 15.2 mm
- net /IO7: track 0.00 -> 12.7 mm
- net /IO6: track 0.00 -> 12.7 mm
- net /IO11: track 0.00 -> 10.2 mm
- net /IO10: track 0.00 -> 10.2 mm
- net unconnected-(J17-Pin_2-Pad2): track 0.00 -> 5.10 mm, vias 0 -> 1
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