File: KiCad/Protection_Catapult_PCB/Protection_Catapult_PCB.kicad_pcb (KiCad board)
At the start: 2 copper layers, 160 x 100 mm, 21 parts, among them J1 Motor_I, J2 Motor_D, J3 Control_D, J4 Control_I, J5 Alimentacion, J6 Alimentacion 5V, U1 A4988_STEPPER_MOTOR_DRIVER_CA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, U2 A4988_STEPPER_MOTOR_DRIVER_CA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, U3 DC_DC_small

Commit message: PCB Update.
Parts:
- added C1: C, Capacitor_THT:C_Disc_D4.3mm_W1.9mm_P5.00mm, F.Cu at (96.6, 132.1)
- added C2: C, Capacitor_THT:C_Disc_D4.3mm_W1.9mm_P5.00mm, F.Cu at (83.7, 106.7)
- added J10: Screw_Terminal_01x03, Connector_JST:JST_XH_B3B-XH-A_1x03_P2.50mm_Vertical, F.Cu at (116.8, 109.3)
- added J11: Motor NEMA I, Connector_JST:JST_XH_B2B-XH-A_1x02_P2.50mm_Vertical, F.Cu at (213.8, 49.1)
- added J12: Motor DC, Connector_JST:JST_XH_B2B-XH-A_1x02_P2.50mm_Vertical, F.Cu at (213.8, 56.9)
- added J13: Motores 28BYJ-48, Connector_JST:JST_XH_B4B-XH-A_1x04_P2.50mm_Vertical, F.Cu at (213.8, 72.5)
- added J15: Servo, Connector_JST:JST_XH_B1B-XH-AM_1x01_P2.50mm_Vertical, F.Cu at (213.8, 80.3)
- added J16: Motor NEMA D, Connector_JST:JST_XH_B2B-XH-A_1x02_P2.50mm_Vertical, F.Cu at (213.8, 64.7)
- added J7: Screw_Terminal_01x05, Connector_JST:JST_XH_B5B-XH-A_1x05_P2.50mm_Vertical, F.Cu at (109.2, 119.2)
- added J8: Screw_Terminal_01x05, Connector_JST:JST_XH_B5B-XH-A_1x05_P2.50mm_Vertical, F.Cu at (73.7, 111.8)
- added J9: Screw_Terminal_01x04, Connector_JST:JST_XH_B4B-XH-A_1x04_P2.50mm_Vertical, F.Cu at (91.4, 119.3)
- added U4: ULN2003A, Package_DIP:CERDIP-16_W7.62mm_SideBrazed, F.Cu at (96.6, 111.8)
- added U5: ULN2003A, Package_DIP:CERDIP-16_W7.62mm_SideBrazed, F.Cu at (86.4, 127.0)
- added U6: ESP32-S3-DevKitC, PCM_Espressif:ESP32-S3-DevKitC, F.Cu at (185.4, 53.3)
Routing:
- net +12V: track 91.7 -> 241.8 mm
- net GND: track 279.4 -> 322.7 mm, vias 9 -> 13
- net /In4: track 0.00 -> 10.3 mm
- net /In3: track 0.00 -> 10.2 mm
- net /In2: track 0.00 -> 10.2 mm
- net /In1: track 0.00 -> 10.2 mm
- net Net-(J7-Pin_1): track 0.00 -> 5.24 mm
- net Net-(J8-Pin_1): track 0.00 -> 5.13 mm
- net Net-(J8-Pin_2): track 0.00 -> 5.11 mm
- net Net-(J8-Pin_3): track 0.00 -> 5.10 mm
- net Net-(J7-Pin_3): track 0.00 -> 5.09 mm
- net Net-(J8-Pin_4): track 0.00 -> 5.08 mm
- net Net-(J7-Pin_2): track 0.00 -> 5.05 mm
- net Net-(J7-Pin_4): track 0.00 -> 5.02 mm
- net (no net): vias 1220 -> 970

Commit message: NEMA 17 supports added.
Parts:
- removed U6: ESP32-S3-DevKitC, PCM_Espressif:ESP32-S3-DevKitC
- added J14: Screw_Terminal_01x09, Connector_PinHeader_2.54mm:PinHeader_1x09_P2.54mm_Vertical, F.Cu at (160.0, 48.3)
- added J17: Motor, Connector_JST:JST_XH_B2B-XH-A_1x02_P2.50mm_Vertical, F.Cu at (119.4, 137.2)
- added J18: Screw_Terminal_01x09, Connector_PinHeader_2.54mm:PinHeader_1x09_P2.54mm_Vertical, F.Cu at (175.3, 48.3)
- J10: value Screw_Terminal_01x03 -> Servo
- J12: footprint Connector_JST:JST_XH_B2B-XH-A_1x02_P2.50mm_Vertical -> Connector_JST:JST_XH_B4B-XH-A_1x04_P2.50mm_Vertical
- J15: value Servo -> Final carrera; footprint Connector_JST:JST_XH_B1B-XH-AM_1x01_P2.50mm_Vertical -> Connector_JST:JST_XH_B2B-XH-A_1x02_P2.50mm_Vertical
- moved J15 56.5 mm to (157.5, 76.2), turned to 180 degrees
- moved J10 52.9 mm to (147.3, 66.0)
- moved J13 41.4 mm to (172.6, 76.2), turned to 180 degrees
- moved J12 35.8 mm to (185.4, 78.7), turned to 90 degrees
- moved J11 28.7 mm to (185.4, 53.3), turned to 90 degrees
- moved J16 28.4 mm to (185.4, 63.5), turned to 90 degrees
Connections:
- J10 pad 1: /Servo -> /IO6
- J11 pad 1: Net-(J11-Pin_1) -> /IO12
- J11 pad 2: Net-(J11-Pin_2) -> /IO13
- J12 pad 1: Net-(J12-Pin_1) -> GND
- J12 pad 2: Net-(J12-Pin_2) -> /IO8
- J13 pad 1: Net-(J13-Pin_1) -> /IO2
- J13 pad 2: Net-(J13-Pin_2) -> /IO3
- J13 pad 3: Net-(J13-Pin_3) -> /IO4
- J13 pad 4: Net-(J13-Pin_4) -> /IO5
- J15 pad 1: Net-(J15-Pin_1) -> GND
- J16 pad 1: Net-(J16-Pin_1) -> /IO10
- J16 pad 2: Net-(J16-Pin_2) -> /IO11
Routing:
- net GND: track 322.7 -> 409.2 mm
- net +5V: track 195.8 -> 277.1 mm, vias 6 -> 16
- net /IO2: track 0.00 -> 33.1 mm
- net /IO3: track 0.00 -> 28.0 mm
- net /IO4: track 0.00 -> 22.9 mm
- net /IO9: track 0.00 -> 17.9 mm
- net /IO8: track 0.00 -> 17.8 mm
- net /IO5: track 0.00 -> 17.8 mm
- net /IO12: track 0.00 -> 15.2 mm
- net /IO13: track 0.00 -> 15.2 mm
- net /IO7: track 0.00 -> 12.7 mm
- net /IO6: track 0.00 -> 12.7 mm
- net /IO11: track 0.00 -> 10.2 mm
- net /IO10: track 0.00 -> 10.2 mm
- net unconnected-(J17-Pin_2-Pad2): track 0.00 -> 5.10 mm, vias 0 -> 1
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
Commit message: Enable for A4988 PCB update toi disconect the motors.
Parts:
- added J19: Screw_Terminal_01x01, Connector_PinHeader_2.54mm:PinHeader_1x01_P2.54mm_Vertical, F.Cu at (134.6, 83.8)
- added J20: Screw_Terminal_01x01, Connector_PinHeader_2.54mm:PinHeader_1x01_P2.54mm_Vertical, F.Cu at (154.9, 53.3)
Connections:
- U1 pad 1: unconnected-(U1-~{ENABLE}-Pad1) -> /Enable
- U2 pad 1: unconnected-(U2-~{ENABLE}-Pad1) -> /Enable
Routing:
- net /Enable: track 0.00 -> 68.6 mm, vias 0 -> 2
- net (no net): vias 1018 -> 993
